Commit message: add blender files and link models

File: models/rocket_model.urdf (robot description, URDF)
Before this commit: robot rocket, 3 links, 2 joints
Links:
- added link fins_visual, mass 0.0001; visual mesh filename=rocket_fins.obj scale=1 1 1
- added link main_body_visual, mass 0.0001; visual mesh filename=rocket_main_body.obj scale=1 1 1
- added link nozzle_visual, mass 0.0001; visual mesh filename=rocket_nozzle.obj scale=1 1 1
Joints:
- added joint fins_visual_joint: type fixed, parent base_link, child fins_visual, origin xyz=0.0 0.0 0.0 rpy=0.0 0.0 0.0
- added joint main_body_visual_joint: type fixed, parent base_link, child main_body_visual, origin xyz=0.0 0.0 0.0 rpy=0.0 0.0 0.0
- added joint nozzle_visual_joint: type fixed, parent base_link, child nozzle_visual, origin xyz=0.0 0.0 0.0 rpy=0.0 0.0 0.0
